File: PCB_design/PCB_robot_controller/NUCLEO64-F401RE.kicad_sch (KiCad schematic)
At the start: 7 parts, among them J3 Conn_02x19_Odd_Even, J4 Conn_02x19_Odd_Even, U1 L7805

Commit message: pcb to production
Parts:
- U1: value L7805 -> L7812; footprint Package_TO_SOT_THT:TO-220-3_Vertical -> Package_TO_SOT_THT:TO-220-3_Horizontal_TabDown
Connections:
- net +5V: no longer C3.1, J3.24 (Pin_24), U1.3 (OUT)
- net DIR_1: now also J4.12 (Pin_12); no longer J4.4 (Pin_4)
- net DIR_2: now also J4.26 (Pin_26); no longer J4.28 (Pin_28)
- net LS_1: now also J4.16 (Pin_16); no longer J4.6 (Pin_6)
- net STEP_1: now also J4.14 (Pin_14); no longer J4.2 (Pin_2)
- net STEP_2: now also J4.28 (Pin_28); no longer J4.26 (Pin_26)
- net AGND: no longer names the net of J4.32 (Pin_32)
- net AVDD: no longer names the net of J4.7 (Pin_7)
- net E5V: no longer names the net of J3.6 (Pin_6)
- net EN renamed PC9
- removed net GPIO: J3.28 (Pin_28), J3.3 (Pin_3), J3.30 (Pin_30), J3.32 (Pin_32), J3.34 (Pin_34), J3.36 (Pin_36), J3.37 (Pin_37), J4.12 (Pin_12), J4.13 (Pin_13), J4.14 (Pin_14), J4.15 (Pin_15), J4.16 (Pin_16), J4.17 (Pin_17), J4.19 (Pin_19), J4.21 (Pin_21), J4.22 (Pin_22), J4.23 (Pin_23), J4.24 (Pin_24), J4.25 (Pin_25), J4.27 (Pin_27), J4.29 (Pin_29), J4.3 (Pin_3), J4.5 (Pin_5)
- net U5V: no longer names the net of J4.8 (Pin_8)
- net VDD: no longer names the net of J3.33 (Pin_33)
- net VDD: no longer J3.5 (Pin_5)
- new net +12V: C3.1, J3.24 (Pin_24), U1.3 (OUT)
- new net EN_1: J4.6 (Pin_6)
- new net EN_2: J4.24 (Pin_24)
- new net EN_3: J3.3 (Pin_3)
- new net EN_4: J3.37 (Pin_37)
- new net PA0: J3.28 (Pin_28)
- new net PA1: J3.30 (Pin_30)
- new net PA4: J3.32 (Pin_32)
- new net PA6: J4.13 (Pin_13)
- new net PA7: J4.15 (Pin_15)
- new net PA9: J4.21 (Pin_21)
- new net PB0: J3.34 (Pin_34)
- new net PB2: J4.22 (Pin_22)
- new net PB6: J4.17 (Pin_17)
- new net PB8: J4.3 (Pin_3)
- new net PB9: J4.5 (Pin_5)
- new net PC1: J3.36 (Pin_36)
- new net PC6: J4.4 (Pin_4)
- new net PC7: J4.19 (Pin_19)
- new net PC8: J4.2 (Pin_2)
- new net SW_F1: J4.23 (Pin_23)
- new net SW_F2: J4.25 (Pin_25)
- new net SW_F3: J4.27 (Pin_27)
- new net SW_F4: J4.29 (Pin_29)
- no-connect marks 17 -> 42
Other:
- note added: "NRST and BOOT0 are already on the NUCLEO64 board"
