File: PCB_design/PCB_robot_controller/PCB_robot_controller.kicad_pcb (KiCad board)
At the start: 2 copper layers, 22 parts, among them J3 Conn_02x19_Odd_Even, J4 Conn_02x19_Odd_Even, Q1 IRF6710S2, U1 L7805, U2 MAX485E

Commit message: pcb to production
Parts:
- added C4: 100nF, Capacitor_SMD:C_0805_2012Metric, F.Cu at (144.7, 135.3)
- added C5: 100nF, Capacitor_SMD:C_0805_2012Metric, F.Cu at (158.0, 135.3)
- added C6: 100nF, Capacitor_SMD:C_0805_2012Metric, F.Cu at (171.0, 135.3)
- added C7: 100nF, Capacitor_SMD:C_0805_2012Metric, F.Cu at (183.2, 135.3)
- added R6: 10K, Resistor_SMD:R_0805_2012Metric, F.Cu at (177.1, 135.3)
- added R7: 120, Resistor_SMD:R_0805_2012Metric, F.Cu at (188.2, 72.0)
- added SW1: SW_Push, Button_Switch_THT:SW_PUSH_6mm_H5mm, F.Cu at (144.9, 142.8)
- added SW2: SW_Push, Button_Switch_THT:SW_PUSH_6mm_H5mm, F.Cu at (158.2, 142.8)
- added SW3: SW_Push, Button_Switch_THT:SW_PUSH_6mm_H5mm, F.Cu at (171.2, 142.8)
- added SW4: SW_Push, Button_Switch_THT:SW_PUSH_6mm_H5mm, F.Cu at (183.4, 142.8)
- Q1: footprint Package_TO_SOT_THT:TO-220-3_Vertical -> Package_TO_SOT_THT:TO-220-3_Horizontal_TabDown
- U1: value L7805 -> L7812; footprint Package_TO_SOT_THT:TO-220-3_Vertical -> Package_TO_SOT_THT:TO-220-3_Horizontal_TabDown
- moved COM 103.5 mm to (204.8, 73.7), turned to 90 degrees
- moved MOTOR3 103.4 mm to (115.4, 82.3), turned to -90 degrees
- moved POWER 83.3 mm to (115.4, 71.3), turned to -90 degrees
- moved U1 79.8 mm to (144.2, 72.2), turned to -90 degrees
- moved D2 76.7 mm to (128.1, 71.3), turned to 180 degrees
- moved C2 71.6 mm to (139.5, 72.3), turned to -90 degrees
- moved C1 70.0 mm to (184.0, 70.0), turned to 0 degrees
- moved C3 63.5 mm to (139.5, 77.0), turned to 90 degrees
- moved U2 57.2 mm to (176.8, 72.0), turned to 0 degrees
- moved GRIPPER 50.9 mm to (115.4, 131.8)
- moved Q1 49.5 mm to (145.5, 116.8), turned to 0 degrees
- moved D1 44.5 mm to (127.5, 132.8)
- moved R2 35.4 mm to (150.6, 122.3), turned to 90 degrees
- moved R1 33.8 mm to (148.0, 122.3), turned to 90 degrees
- moved MOTOR2 24.4 mm to (204.7, 123.3)
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- renumbered RS485 to COM, GRIPPER1 to GRIPPER, POWER1 to POWER
Connections:
- C3 pad 1: +5V -> +12V
- J3 pad 24: +5V -> +12V
- J3 pad 28: GPIO -> /NUCLEO64-F401RE/PA0
- J3 pad 3: GPIO -> EN_3
- J3 pad 30: GPIO -> /NUCLEO64-F401RE/PA1
- J3 pad 32: GPIO -> /NUCLEO64-F401RE/PA4
- J3 pad 33: VDD -> unconnected-(J3-Pin_33-Pad33)
- J3 pad 34: GPIO -> /NUCLEO64-F401RE/PB0
- J3 pad 36: GPIO -> /NUCLEO64-F401RE/PC1
- J3 pad 37: GPIO -> EN_4
- J3 pad 5: VDD -> unconnected-(J3-Pin_5-Pad5)
- J3 pad 6: E5V -> unconnected-(J3-Pin_6-Pad6)
- J4 pad 1: EN -> /NUCLEO64-F401RE/PC9
- J4 pad 12: GPIO -> DIR_1
- J4 pad 13: GPIO -> /NUCLEO64-F401RE/PA6
- J4 pad 14: GPIO -> STEP_1
- J4 pad 15: GPIO -> /NUCLEO64-F401RE/PA7
- J4 pad 16: GPIO -> LS_1
- J4 pad 17: GPIO -> /NUCLEO64-F401RE/PB6
- J4 pad 19: GPIO -> /NUCLEO64-F401RE/PC7
- J4 pad 2: STEP_1 -> /NUCLEO64-F401RE/PC8
- J4 pad 21: GPIO -> /NUCLEO64-F401RE/PA9
- J4 pad 22: GPIO -> /NUCLEO64-F401RE/PB2
- J4 pad 23: GPIO -> SW_F1
- J4 pad 24: GPIO -> EN_2
- J4 pad 25: GPIO -> SW_F2
- J4 pad 26: STEP_2 -> DIR_2
- J4 pad 27: GPIO -> SW_F3
- J4 pad 28: DIR_2 -> STEP_2
- J4 pad 29: GPIO -> SW_F4
- J4 pad 3: GPIO -> /NUCLEO64-F401RE/PB8
- J4 pad 32: AGND -> unconnected-(J4-Pin_32-Pad32)
- J4 pad 4: DIR_1 -> /NUCLEO64-F401RE/PC6
- J4 pad 5: GPIO -> /NUCLEO64-F401RE/PB9
- J4 pad 6: LS_1 -> EN_1
- J4 pad 7: AVDD -> unconnected-(J4-Pin_7-Pad7)
- J4 pad 8: U5V -> unconnected-(J4-Pin_8-Pad8)
- MOTOR1 pad 1: VDD -> +5V
- MOTOR1 pad 5: EN -> EN_1
- MOTOR2 pad 1: VDD -> +5V
- MOTOR2 pad 5: EN -> EN_2
- MOTOR3 pad 1: VDD -> +5V
- MOTOR3 pad 5: EN -> EN_3
- MOTOR4 pad 1: VDD -> +5V
- MOTOR4 pad 5: EN -> EN_4
- U1 pad 3: +5V -> +12V
Routing:
- net GND: track 5.43 -> 396.4 mm, vias 0 -> 4
- net +5V: track 5.36 -> 323.4 mm
- net +24V: track 7.11 -> 98.5 mm, vias 0 -> 2
- net SW_F1: track 0.00 -> 69.5 mm
- net USART_RX: track 0.00 -> 69.4 mm, vias 0 -> 1
- net SW_F2: track 0.00 -> 63.1 mm
- net USART_TX: track 0.00 -> 60.5 mm, vias 0 -> 1
- net USART_DE: track 1.27 -> 60.1 mm, vias 0 -> 1
- net SW_F3: track 0.00 -> 49.5 mm
- net +12V: track 0.00 -> 43.6 mm, vias 0 -> 2
- net /robot_control/GRIPPER -: track 0.00 -> 38.2 mm
- net SW_F4: track 0.00 -> 36.8 mm
- net GRIPPER: track 0.00 -> 31.9 mm, vias 0 -> 1
- net LS_3: track 0.00 -> 24.6 mm
- net EN_3: track 0.00 -> 24.2 mm
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- added copper zone on B.Cu, net GND
- added copper zone on F.Cu, net GND
Other:
- board outline added: 106 x 88 mm
- board text added: "+"
- board text added: "+24V"
- board text added: "+5V LS STEP DIR EN GND"
- board text added: "-"
- board text added: "GND"
- board text added: "RS485-A"
- board text added: "RS485-B"
