File: PCB_design/PCB_robot_controller/robot_control.kicad_sch (KiCad schematic)
At the start: 9 parts, among them Q1 IRF6710S2

Commit message: pcb to production
Parts:
- Q1: footprint Package_TO_SOT_THT:TO-220-3_Vertical -> Package_TO_SOT_THT:TO-220-3_Horizontal_TabDown
Connections:
- removed net EN: MOTOR1.5 (Pin_5), MOTOR2.5 (Pin_5), MOTOR3.5 (Pin_5), MOTOR4.5 (Pin_5)
- net VDD renamed +5V
- new net EN_1: MOTOR1.5 (Pin_5)
- new net EN_2: MOTOR2.5 (Pin_5)
- new net EN_3: MOTOR3.5 (Pin_5)
- new net EN_4: MOTOR4.5 (Pin_5)
